Commit message: Checkpoint 8: Multi-robot spawn and TF-based robot chase working

File: barista_robot_description/urdf/barista_robot_model.urdf (robot description, URDF)
Before this commit: robot barista_robot, 10 links, 9 joints
Links:
- removed link laser_link
- removed link standoff_1
- removed link standoff_2
- removed link standoff_3
- removed link standoff_4
- link base_link: mass 8.0 -> 5.0; geometry collision cylinder length=0.1 radius=0.18; visual cylinder length=0.1 radius=0.18
- link caster_wheel: geometry visual sphere radius=0.03
- link left_wheel: geometry visual cylinder length=0.02 radius=0.05
- link right_wheel: geometry visual cylinder length=0.02 radius=0.05
Joints:
- removed joint caster_joint
- removed joint laser_joint
- removed joint standoff_1_joint
- removed joint standoff_2_joint
- removed joint standoff_3_joint
- removed joint standoff_4_joint
- added joint caster_wheel_joint: type fixed, parent base_link, child caster_wheel, origin xyz=-0.15 0 0.02 rpy=0 0 0
- joint left_wheel_joint: origin xyz=0 0.18 0.0352 rpy=0 1.5708 0 -> xyz=0 0.18 0.025 rpy=0 1.5707 0
- joint right_wheel_joint: origin xyz=0 -0.18 0.0352 rpy=0 1.5708 0 -> xyz=0 -0.18 0.025 rpy=0 1.5707 0
- joint top_plate_joint: origin xyz=0 0 0.355 -> xyz=0 0 0.1 rpy=0 0 0
